Commit message: add a f/t snesor and camera

File: end_effectors/franka_hand/franka_hand_arguments.xacro (robot description, xacro)
@@ -14,5 +14,6 @@
   <xacro:arg name="xyz_ee" default="0 0 0" />
   <!-- Rotation offset between ee and parent frame -->
-  <xacro:arg name="rpy_ee" default= "0 0 ${-pi/4}" />
+  <!-- <xacro:arg name="rpy_ee" default= "0 0 ${-pi/4}" /> -->
+  <xacro:arg name="rpy_ee" default= "${-pi/2} 0 ${pi}" />
   <!-- Position offset between ee frame and tcp frame -->
   <xacro:arg name="tcp_xyz" default="0 0 0.1034" />

File: robots/common/franka_robot.xacro (robot description, xacro)
@@ -53,6 +53,15 @@
       <xacro:property name="special_connection" value="$(arg special_connection)" />
       <xacro:property name="connection" value="${special_connection if special_connection != '' else arm_id + '_link8'}" />
+      <!-- F/T sensor and camera -->
+      <xacro:include filename="$(find franka_description)/end_effectors/sensors/axia80.xacro" />
+      <xacro:axia80 description_pkg="franka_description" parent_link="${arm_prefix_modified}${connection}" child_link="camera_hand"/>
+      <!-- Realsense D455 추가 -->
+      <xacro:include filename="$(find realsense2_description)/urdf/_d435.urdf.xacro"/>
+      <xacro:arg name="use_nominal_extrinsics" default="false"/>
+      <xacro:sensor_d435 parent="camera_hand" name="d435" use_nominal_extrinsics="$(arg use_nominal_extrinsics)">
+        <origin xyz="-0.07 -0.007 -0.033" rpy="${pi/2} 0 -${pi*1/3}"/>
+      </xacro:sensor_d435>
       <xacro:franka_hand
-        connected_to="${arm_prefix_modified}${connection}"
+        connected_to="camera_hand"
         arm_id="${arm_id}"
         arm_prefix="${arm_prefix_modified}"
