Commit message: update

File: end_effectors/sensors/axia80.xacro (robot description, xacro)
@@ -72,5 +72,5 @@
         </inertial>
         <visual>
-            <origin rpy="0 0 0" xyz="0 -0.0 0"/>
+            <origin rpy="0 0 0" xyz="0 -0.0 0.0"/>
             <geometry>
                 <mesh filename="package://franka_description/meshes/robot_ee/sensors/camera_hand.stl" scale="0.001 0.001 0.001"/>
@@ -79,5 +79,5 @@
         </visual>
         <collision>
-        <origin rpy="0 0 0" xyz="0 -0.0 0"/>
+        <origin rpy="0 0 0" xyz="0 -0.0 0.002"/>
         <geometry>
             <mesh filename="package://franka_description/meshes/robot_ee/sensors/camera_hand.stl" scale="0.001 0.001 0.001"/>
@@ -96,5 +96,5 @@
     </joint>
     <joint name="joint_ft_down" type="fixed">
-        <origin rpy="0 0 0" xyz="0.041 0.0 0.041"/>
+        <origin rpy="0 0 0" xyz="0.041 -0.00 0.041"/>
         <parent link="ft_sensor"/>
         <child link="flange_down"/>

File: robots/common/franka_robot.xacro (robot description, xacro)
@@ -57,5 +57,5 @@
       <xacro:axia80 description_pkg="franka_description" parent_link="${arm_prefix_modified}${connection}" child_link="camera_hand"/>
       <!-- Realsense D455 추가 -->
-      <xacro:include filename="$(find realsense2_description)/urdf/_d435.urdf.xacro"/>
+      <xacro:include filename="$(find franka_description)/end_effectors/sensors/_d435.urdf.xacro"/>
       <xacro:arg name="use_nominal_extrinsics" default="false"/>
       <xacro:sensor_d435 parent="camera_hand" name="d435" use_nominal_extrinsics="$(arg use_nominal_extrinsics)">
